File: tuerklingel.sch (EAGLE design)
At the start: 12 parts, among them IC1 ESP-12E/F

Commit message: bauteilbezeichnungen
Parts:
- F1: value (none) -> FSMD020-1210-R
- OK1: value Mosfet -> G3VM41DY1
Changed lines of the file:
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@@
 <part name="C1" library="rcl" deviceset="C-EU" device="C0805" value="0,47u"/>
 <part name="JP3" library="pinhead" deviceset="PINHD-1X5" device=""/>
-<part name="F1" library="resistor" deviceset="R-EU_" device="R1210"/>
-<part name="OK1" library="optocoupler" deviceset="LTV816" device="S" value="Mosfet"/>
+<part name="F1" library="resistor" deviceset="R-EU_" device="R1210" value=" FSMD020-1210-R"/>
+<part name="OK1" library="optocoupler" deviceset="LTV816" device="S" value="G3VM41DY1"/>
 <part name="R1" library="rcl" deviceset="R-EU_" device="R0805" value="1k"/>
 <part name="OK2" library="optocoupler" deviceset="LTV826" device="S"/>
